Commit message: Basic arips gazebo configuration, differential drive, tiltable kinect and lidar, no arm yet

File: arips_description/urdf/arips.urdf (robot description, URDF)
Before this commit: robot arips, 12 links, 11 joints
Links:
- removed link arm_base_link
- removed link camera_link
- removed link gripper_base
- removed link gripper_link_left
- removed link gripper_link_right
- removed link link2
- removed link link3
- removed link link4
- removed link link5
- removed link link6
- removed link tool0
- link base_link: mass None -> 1.5; geometry collision cylinder length=0.15 radius=0.2; visual cylinder length=0.15 radius=0.2
Joints:
- removed joint base_to_right_leg
- removed joint camera_joint
- removed joint gripper_joint
- removed joint gripper_joint_right
- removed joint joint1
- removed joint joint2
- removed joint joint3
- removed joint joint4
- removed joint joint5
- removed joint link6-tool0
- removed joint tool0_gripper

File: arips_description/urdf/arips.urdf.xacro (robot description, xacro)
@@ -1,4 +1,124 @@
 <?xml version="1.0"?>
-<robot name="arips">
+<robot name="arips" xmlns:xacro="http://www.ros.org/wiki/xacro">
+    <xacro:property name="PI" value="3.1415926535897931"/>
+    <xacro:property name="base_height" value="0.15"/>
+    <xacro:property name="base_above_ground" value="0.05"/>
+    <xacro:property name="base_radius" value="0.2"/>
+    <xacro:property name="wheel_base" value="0.34"/>
+    <xacro:property name="wheel_thick" value="0.03"/>
+    <xacro:property name="wheel_radius" value="0.05"/>
+    <xacro:property name="front_wheel_gap" value="0.003"/>
+    <xacro:property name="wheel_damping_factor" value="0.7"/>
+    <xacro:property name="camera_name" value="kinect"/>
+    <gazebo>
+        <plugin name="differential_drive_controller" filename="libgazebo_ros_diff_drive.so">
+            <alwaysOn>true</alwaysOn>
+            <updateRate>50</updateRate>
+            <leftJoint>left_wheel_joint</leftJoint>
+            <rightJoint>right_wheel_joint</rightJoint>
+            <wheelSeparation>${wheel_base}</wheelSeparation>
+            <wheelDiameter>${wheel_radius*2}</wheelDiameter>
+            <torque>5</torque>
+            <commandTopic>cmd_vel</commandTopic>
+            <odometryTopic>odom</odometryTopic>
+            <odometryFrame>odom</odometryFrame>
+            <robotBaseFrame>base_link</robotBaseFrame>
+            <publishWheelTF>true</publishWheelTF>
+            <legacyMode>false</legacyMode>
+        </plugin>
+    </gazebo>
+    <gazebo>
+        <plugin name="gazebo_ros_control" filename="libgazebo_ros_control.so">
+            <robotNamespace>/arips</robotNamespace>
+        </plugin>
+    </gazebo>
+    <gazebo reference="base_link">
+        <sensor type="ray" name="lidar_sensor">
+        <pose>0 0 0.2 0 0 0</pose>
+        <visualize>false</visualize>
+        <update_rate>8</update_rate>
+        <ray>
+            <scan>
+            <horizontal>
+                <samples>360</samples>
+                <resolution>1</resolution>
+                <min_angle>${-PI}</min_angle>
+                <max_angle>${PI}</max_angle>
+            </horizontal>
+            </scan>
+            <range>
+            <min>0.21</min>
+            <max>15.0</max>
+            <resolution>0.01</resolution>
+            </range>
+            <noise>
+            <type>gaussian</type>
+            <!-- Noise parameters based on published spec for Hokuyo laser
+                achieving "+-30mm" accuracy at range < 10m.  A mean of 0.0m and
+                stddev of 0.01m will put 99.7% of samples within 0.03m of the true
+                reading. -->
+            <mean>0.0</mean>
+            <stddev>0.02</stddev>
+            </noise>
+        </ray>
+        <plugin name="gazebo_ros_lidar_controller" filename="libgazebo_ros_laser.so">
+            <topicName>/base_scan</topicName>
+            <frameName>base_link</frameName>
+        </plugin>
+        </sensor>
+    </gazebo>
+      <gazebo reference="base_link">
+        <mu1>0.0</mu1>
+        <mu2>0.0</mu2>
+    </gazebo>
+    <gazebo reference="left_wheel">
+        <mu1>0.8</mu1>
+        <mu2>0.8</mu2>
+    </gazebo>
+    <gazebo reference="right_wheel">
+        <mu1>0.8</mu1>
+        <mu2>0.8</mu2>
+    </gazebo>
+    <gazebo reference="kinect_link">
+        <sensor name="kinect_camera" type="depth">
+            <update_rate>20</update_rate>
+            <camera>
+            <horizontal_fov>1.047198</horizontal_fov>
+            <image>
+                <width>320</width>
+                <height>480</height>
+                <format>R8G8B8</format>
+            </image>
+            <clip>
+                <near>0.04</near>
+                <far>8</far>
+            </clip>
+            </camera>
+            <plugin name="kinect_plugin" filename="libgazebo_ros_openni_kinect.so">
+            <baseline>0.2</baseline>
+            <alwaysOn>true</alwaysOn>
+            <updateRate>0</updateRate>
+            <cameraName>${camera_name}_ir</cameraName>
+            <imageTopicName>/${camera_name}/color/image_raw</imageTopicName>
+            <cameraInfoTopicName>/${camera_name}/color/camera_info</cameraInfoTopicName>
+            <depthImageTopicName>/${camera_name}/depth/image_raw</depthImageTopicName>
+            <depthImageInfoTopicName>/${camera_name}/depth/camera_info</depthImageInfoTopicName>
+            <pointCloudTopicName>/${camera_name}/depth/points</pointCloudTopicName>
+            <frameName>kinect_link</frameName>
+            <pointCloudCutoff>0.5</pointCloudCutoff>
+            <pointCloudCutoffMax>3.0</pointCloudCutoffMax>
+            <distortionK1>0.00000001</distortionK1>
+            <distortionK2>0.00000001</distortionK2>
+            <distortionK3>0.00000001</distortionK3>
+            <distortionT1>0.00000001</distortionT1>
+            <distortionT2>0.00000001</distortionT2>
+            <CxPrime>0</CxPrime>
+            <Cx>0</Cx>
+            <Cy>0</Cy>
+            <focalLength>0</focalLength>
+            <hackBaseline>0</hackBaseline>
+            </plugin>
+        </sensor>
+    </gazebo>
   <link name="base_link">
     <visual>
@@ -8,6 +128,93 @@
       <origin rpy="0 0 -1.57075"/>
     </visual>
-  </link>
-  <link name="camera_link">
+    <!-- rear wheel
+    <visual>
+     <geometry>
+            <sphere radius="${wheel_radius}"/>
+        </geometry>
+        <origin xyz="${-base_radius + wheel_radius} 0 ${wheel_radius}" rpy="0 0 0"/>
+    </visual>
+    -->
+    <collision>
+        <geometry>
+            <cylinder radius="${base_radius}" length="${base_height}"/>
+        </geometry>
+        <origin xyz="0 0 ${base_height/2 + base_above_ground}" rpy="0 0 0"/>
+    </collision>
+    <collision>
+        <geometry>
+            <sphere radius="${wheel_radius}"/>
+        </geometry>
+        <origin xyz="${-base_radius + wheel_radius + 0.001} 0 ${wheel_radius}" rpy="0 0 0"/>
+    </collision>
+    <collision>
+        <geometry>
+            <sphere radius="${wheel_radius}"/>
+        </geometry>
+        <origin xyz="${base_radius - wheel_radius - 0.001} 0 ${wheel_radius + front_wheel_gap}" rpy="0 0 0"/>
+    </collision>
+    <inertial>
+      <origin xyz="-0.05 0 ${base_height/2 + base_above_ground}" rpy="0 0 0"/>
+      <mass value="1.5"/>
+      <inertia ixx="0.01625" ixy="0.0" ixz="0.0" iyy="0.01625" iyz="0.0" izz="0.03"/>
+    </inertial>
+  </link>
+  <link name="right_wheel">
+      <!--
+    <visual>
+      <origin rpy="0 0 0" xyz="0 0 0"/>
+      <geometry>
+        <cylinder length="${wheel_thick}" radius="${wheel_radius}"/>
+      </geometry>
+    </visual>
+      -->
+    <collision>
+      <origin rpy="0 0 0" xyz="0 0 0"/>
+      <geometry>
+        <cylinder length="${wheel_thick}" radius="${wheel_radius}"/>
+      </geometry>
+    </collision>
+    <inertial>
+      <origin xyz="0 0 0" rpy="0 0 0"/>
+      <mass value="0.2"/>
+      <inertia ixx="0.0007" ixy="0.0" ixz="0.0" iyy="0.0007" iyz="0.0" izz="0.00125"/>
+    </inertial>
+  </link>
+  <joint name="right_wheel_joint" type="continuous">
+    <parent link="base_link"/>
+    <child link="right_wheel"/>
+    <axis xyz="0 0 1"/>
+    <origin xyz="0 -${wheel_base/2} ${wheel_radius}" rpy="${-PI/2} 0 0"/>
+    <dynamics damping="${wheel_damping_factor}"/>
+  </joint>
+  <link name="left_wheel">
+      <!--
+    <visual>
+      <origin rpy="0 0 0" xyz="0 0 0"/>
+      <geometry>
+        <cylinder length="${wheel_thick}" radius="${wheel_radius}"/>
+      </geometry>
+    </visual>
+      -->
+    <collision>
+      <origin rpy="0 0 0" xyz="0 0 0"/>
+      <geometry>
+        <cylinder length="${wheel_thick}" radius="${wheel_radius}"/>
+      </geometry>
+    </collision>
+    <inertial>
+      <origin xyz="0 0 0" rpy="0 0 0"/>
+      <mass value="0.2"/>
+      <inertia ixx="0.0007" ixy="0.0" ixz="0.0" iyy="0.0007" iyz="0.0" izz="0.00125"/>
+    </inertial>
+  </link>
+  <joint name="left_wheel_joint" type="continuous">
+    <parent link="base_link"/>
+    <child link="left_wheel"/>
+    <axis xyz="0 0 1"/>
+    <origin xyz="0 ${wheel_base/2} ${wheel_radius}" rpy="${-PI/2} 0 0"/>
+    <dynamics damping="${wheel_damping_factor}"/>
+  </joint>
+  <link name="kinect_link">
     <visual>
       <geometry>
@@ -15,13 +222,36 @@
       </geometry>
     </visual>
-  </link>
-  <joint name="camera_joint" type="revolute">
-  <limit effort="1000.0" lower="-1" upper="1" velocity="0.5"/>
-    <parent link="base_link"/>
-    <child link="camera_link"/>
+    <collision>
+      <origin rpy="0 0 0" xyz="0 0 0"/>
+      <geometry>
+        <box size="0.06 0.2 0.03"/>
+      </geometry>
+    </collision>
+    <inertial>
+      <origin xyz="0 0 0" rpy="0 0 0"/>
+      <mass value="0.2"/>
+      <inertia ixx="0.0007" ixy="0.0" ixz="0.0" iyy="0.0007" iyz="0.0" izz="0.00125"/>
+    </inertial>
+  </link>
+  <joint name="kinect_joint" type="revolute">
+    <limit effort="10.0" lower="-1" upper="1" velocity="0.2"/>
+    <parent link="base_link"/>
+    <child link="kinect_link"/>
     <origin xyz="-0.14 0 0.74" rpy="0 0 0"/>
     <axis xyz="0 1 0" />
-  </joint>
-  <joint name="base_to_right_leg" type="fixed">
+    <dynamics damping="0.07"/>
+  </joint>
+  <transmission name="kinect_trans">
+    <type>transmission_interface/SimpleTransmission</type>
+    <joint name="kinect_joint">
+      <hardwareInterface>hardware_interface/EffortJointInterface</hardwareInterface>
+    </joint>
+    <actuator name="kinect_motor">
+      <hardwareInterface>hardware_interface/EffortJointInterface</hardwareInterface>
+      <mechanicalReduction>1</mechanicalReduction>
+    </actuator>
+  </transmission>
+    <!--
+  <joint name="base_to_arm" type="fixed">
     <parent link="base_link"/>
     <child link="arm_base_link"/>
@@ -29,3 +259,4 @@
   </joint>
   <include filename="$(find arips_arm_description)/urdf/arips_arm.xacro" />
+  -->
 </robot>
