Commit message: Updated gmapping parameters and arips_description to fit

File: arips_description/urdf/arips.urdf.xacro (robot description, xacro)
@@ -9,5 +9,5 @@
     <xacro:property name="wheel_radius" value="0.05"/>
     <xacro:property name="front_wheel_gap" value="0.003"/>
-    <xacro:property name="wheel_damping_factor" value="0.7"/>
+    <xacro:property name="wheel_damping_factor" value="0.2"/>
     <xacro:property name="camera_name" value="kinect"/>
     <gazebo>
@@ -23,7 +23,9 @@
             <odometryTopic>odom</odometryTopic>
             <odometryFrame>odom</odometryFrame>
-            <robotBaseFrame>base_link</robotBaseFrame>
+            <robotBaseFrame>arips_base</robotBaseFrame>
             <publishWheelTF>true</publishWheelTF>
+            <publishTf>false</publishTf>
             <legacyMode>false</legacyMode>
+            <odometrySource>encoder</odometrySource>
         </plugin>
     </gazebo>
@@ -33,5 +35,5 @@
         </plugin>
     </gazebo>
-    <gazebo reference="base_link">
+    <gazebo reference="arips_base">
         <sensor type="ray" name="lidar_sensor">
         <pose>0 0 0.2 0 0 0</pose>
@@ -63,20 +65,21 @@
         </ray>
         <plugin name="gazebo_ros_lidar_controller" filename="libgazebo_ros_laser.so">
-            <topicName>/base_scan</topicName>
-            <frameName>base_link</frameName>
+            <topicName>/scan</topicName>
+            <frameName>arips_base</frameName>
         </plugin>
         </sensor>
     </gazebo>
-      <gazebo reference="base_link">
-        <mu1>0.0</mu1>
-        <mu2>0.0</mu2>
-    </gazebo>
+      <gazebo reference="arips_base">
+        <mu1>0.0001</mu1>
+        <mu2>0.0001</mu2>
+    </gazebo>
+    <!-- Use slightly different friction for individual wheels to be more realistic -->
     <gazebo reference="left_wheel">
-        <mu1>0.8</mu1>
-        <mu2>0.8</mu2>
+        <mu1>0.81</mu1>
+        <mu2>0.81</mu2>
     </gazebo>
     <gazebo reference="right_wheel">
-        <mu1>0.8</mu1>
-        <mu2>0.8</mu2>
+        <mu1>0.81</mu1>
+        <mu2>0.81</mu2>
     </gazebo>
     <gazebo reference="kinect_link">
@@ -87,10 +90,10 @@
             <image>
                 <width>320</width>
-                <height>480</height>
+                <height>240</height>
                 <format>R8G8B8</format>
             </image>
             <clip>
                 <near>0.04</near>
-                <far>8</far>
+                <far>25</far>
             </clip>
             </camera>
@@ -121,5 +124,5 @@
         </sensor>
     </gazebo>
-  <link name="base_link">
+  <link name="arips_base">
     <visual>
       <geometry>
@@ -182,5 +185,5 @@
   </link>
   <joint name="right_wheel_joint" type="continuous">
-    <parent link="base_link"/>
+    <parent link="arips_base"/>
     <child link="right_wheel"/>
     <axis xyz="0 0 1"/>
@@ -210,5 +213,5 @@
   </link>
   <joint name="left_wheel_joint" type="continuous">
-    <parent link="base_link"/>
+    <parent link="arips_base"/>
     <child link="left_wheel"/>
     <axis xyz="0 0 1"/>
@@ -236,5 +239,5 @@
   <joint name="kinect_joint" type="revolute">
     <limit effort="10.0" lower="-1" upper="1" velocity="0.2"/>
-    <parent link="base_link"/>
+    <parent link="arips_base"/>
     <child link="kinect_link"/>
     <origin xyz="-0.14 0 0.74" rpy="0 0 0"/>
@@ -254,6 +257,6 @@
     <!--
   <joint name="base_to_arm" type="fixed">
-    <parent link="base_link"/>
-    <child link="arm_base_link"/>
+    <parent link="arips_base"/>
+    <child link="arm_arips_base"/>
     <origin rpy="-0.028 0 0" xyz="0.163 -0.006 0.055"/>
   </joint>
