Commit message: [arips_arm_description] Basic arips arm urdf model

File: arips_arm_description/urdf/arips_arm.urdf (robot description, URDF)
Before this commit: robot multipleshapes, 2 links, 1 joints
Links:
- removed link right_leg
- added link link2; visual cylinder length=0.07 radius=0.025
- added link link3; visual box size=0.02 0.05 0.12
- added link link4; visual box size=0.02 0.04 0.15
- added link link5; visual box size=0.01 0.04 0.03
- added link link6; visual cylinder length=0.025 radius=0.01
- link base_link: geometry visual box size=0.05 0.05 0.01
Joints:
- removed joint base_to_right_leg
- added joint joint1: type continuous, parent base_link, child link2, origin xyz=0 0 0.01, axis 0 0 1
- added joint joint2: type continuous, parent link2, child link3, origin xyz=0 0 0.07, axis 0 1 0
- added joint joint3: type continuous, parent link3, child link4, origin xyz=0 0 0.12, axis 0 1 0
- added joint joint4: type continuous, parent link4, child link5, origin xyz=0 0 0.15, axis 0 1 0
- added joint joint5: type continuous, parent link5, child link6, origin xyz=0 0 0.015, axis 0 0 1

File: arips_arm_description/urdf/arips_arm.xacro (robot description, xacro)
@@ -1,42 +1,111 @@
 <?xml version="1.0"?>
 <robot name="arips_arm" xmlns:xacro="http://ros.org/wiki/xacro">
-  <xacro:property name="base_height" value="0.7" />
-  <xacro:property name="base_radius" value="0.5" />
+  <material name="white">
+    <color rgba="1 1 1 1"/>
+  </material>
+  <material name="black">
+    <color rgba="0 0 0 1"/>
+  </material>
+  <material name="orange">
+    <color rgba="1 0.6 0 1"/>
+  </material>
+  <xacro:property name="link1_sidelen" value="0.05" />
+  <xacro:property name="link1_height" value="0.01" />
+  <xacro:property name="link2_height" value="0.07" />
+  <xacro:property name="link2_radius" value="0.025" />
+  <xacro:property name="link3_len" value="0.12" />
+  <xacro:property name="link3_thick" value="0.02" />
+  <xacro:property name="link3_width" value="0.05" />
+  <xacro:property name="link4_len" value="0.15" />
+  <xacro:property name="link4_thick" value="0.02" />
+  <xacro:property name="link4_width" value="0.04" />
+  <xacro:property name="link5_len" value="0.03" />
+  <xacro:property name="link5_thick" value="0.01" />
+  <xacro:property name="link5_width" value="0.04" />
+  <xacro:property name="link6_len" value="0.025" />
+  <xacro:property name="link6_radius" value="0.01" />
   <link name="base_link">
   	<visual>
       <geometry>
-        <cylinder length="${base_height}" radius="${base_radius}"/>
+        <box size="${link1_sidelen} ${link1_sidelen} ${link1_height}"/>
       </geometry>
+      <origin xyz="0 0 ${link1_height/2}"/>
+      <material name="black"/>
     </visual>
   </link>
   <link name="link2" >
+  	<visual>
+      <geometry>
+        <cylinder length="${link2_height}" radius="${link2_radius}"/>
+      </geometry>
+      <origin xyz="0 0 ${link2_height/2}"/>
+      <material name="white"/>
+    </visual>
   </link>
   <link name="link3" >
+    <visual>
+      <geometry>
+        <box size="${link3_thick} ${link3_width} ${link3_len}"/>
+      </geometry>
+      <origin xyz="0 0 ${link3_len/2}"/>
+      <material name="white"/>
+    </visual>
   </link>
   <link name="link4" >
+    <visual>
+      <geometry>
+        <box size="${link4_thick} ${link4_width} ${link4_len}"/>
+      </geometry>
+      <origin xyz="0 0 ${link4_len/2}"/>
+      <material name="orange"/>
+    </visual>
   </link>
   <link name="link5" >
+    <visual>
+      <geometry>
+        <box size="${link5_thick} ${link5_width} ${link5_len}"/>
+      </geometry>
+      <origin xyz="0 0 0"/>
+      <material name="orange"/>
+    </visual>
   </link>
   <link name="link6" >
+    <visual>
+      <geometry>
+        <cylinder length="${link6_len}" radius="${link6_radius}"/>
+      </geometry>
+      <origin xyz="0 0 ${link6_len/2}"/>
+      <material name="orange"/>
+    </visual>
   </link>
   <joint name="joint1" type="continuous">
     <parent link="base_link"/>
     <child link="link2"/>
+    <axis xyz="0 0 1"/>
+    <origin xyz="0 0 ${link1_height}"/>
   </joint>
   <joint name="joint2" type="continuous">
     <parent link="link2"/>
     <child link="link3"/>
+    <axis xyz="0 1 0"/>
+    <origin xyz="0 0 ${link2_height}"/>
   </joint>
   <joint name="joint3" type="continuous">
     <parent link="link3"/>
     <child link="link4"/>
+    <axis xyz="0 1 0"/>
+    <origin xyz="0 0 ${link3_len}"/>
   </joint>
   <joint name="joint4" type="continuous">
     <parent link="link4"/>
     <child link="link5"/>
+    <axis xyz="0 1 0"/>
+    <origin xyz="0 0 ${link4_len}"/>
   </joint>
   <joint name="joint5" type="continuous">
     <parent link="link5"/>
     <child link="link6"/>
+    <axis xyz="0 0 1"/>
+    <origin xyz="0 0 ${link5_len / 2}"/>
   </joint>
 </robot>

Commit message: [arips_arm_description] Added tool frame, added moveit config

File: arips_arm_description/urdf/arips_arm.urdf (robot description, URDF)
Before this commit: robot arips_arm, 6 links, 5 joints
Links:
- added link tool0
Joints:
- added joint link6-tool0: type fixed, parent link6, child tool0, origin xyz=0 0 0.025 rpy=0 -1.57075 0

File: arips_arm_description/urdf/arips_arm.xacro (robot description, xacro)
@@ -79,4 +79,6 @@
     </visual>
   </link>
+  <link name="tool0">
+  </link>
   <joint name="joint1" type="continuous">
     <parent link="base_link"/>
@@ -109,3 +111,8 @@
     <origin xyz="0 0 ${link5_len / 2}"/>
   </joint>
+  <joint name="link6-tool0" type="fixed">
+  <parent link="link6" />
+  <child link="tool0" />
+  <origin xyz="0 0 ${link6_len}" rpy="0 -1.57075 0" />
+</joint>
 </robot>

Commit message: [arips_arm] Added gripper to description
Added shitty gripper model to URDF
Fixed joint lengths in ik plugin

File: arips_arm_description/urdf/arips_arm.urdf (robot description, URDF)
Before this commit: robot arips_arm, 7 links, 6 joints
Links:
- added link gripper_base
- added link gripper_link; visual box size=0.05 0.05 0.05
Joints:
- added joint tool0_gripper: type fixed, parent tool0, child gripper_base, origin xyz=0 0 0 rpy=0 0 0
- added joint xgripper_joint: type continuous, parent gripper_base, child gripper_link, origin xyz=0 0 0, axis 0 1 0

File: arips_arm_description/urdf/arips_arm.xacro (robot description, xacro)
@@ -10,4 +10,5 @@
     <color rgba="1 0.6 0 1"/>
   </material>
+  <xacro:property name="pi" value="3.14159265359" />
   <xacro:property name="link1_sidelen" value="0.05" />
   <xacro:property name="link1_height" value="0.01" />
@@ -20,9 +21,10 @@
   <xacro:property name="link4_thick" value="0.02" />
   <xacro:property name="link4_width" value="0.04" />
-  <xacro:property name="link5_len" value="0.03" />
+  <xacro:property name="link5_len" value="0.035" />
   <xacro:property name="link5_thick" value="0.01" />
   <xacro:property name="link5_width" value="0.04" />
-  <xacro:property name="link6_len" value="0.025" />
+  <xacro:property name="link6_len" value="0.085" />
   <xacro:property name="link6_radius" value="0.01" />
+  <xacro:property name="gripper_open_angle" value="0.3" />
   <link name="base_link">
   	<visual>
@@ -73,46 +75,98 @@
     <visual>
       <geometry>
-        <cylinder length="${link6_len}" radius="${link6_radius}"/>
+        <cylinder length="${link6_len-0.04}" radius="${link6_radius}"/>
       </geometry>
-      <origin xyz="0 0 ${link6_len/2}"/>
+      <origin xyz="0 0 ${link6_len/2-0.02}"/>
       <material name="orange"/>
     </visual>
   </link>
   <link name="tool0">
+  <visual>
+      <geometry>
+        <box size="0.012 0.022 0.02"/>
+      </geometry>
+      <origin xyz="-0.04 0 0.02"/>
+      <material name="orange"/>
+    </visual>
   </link>
-  <joint name="joint1" type="continuous">
+  <joint name="joint1" type="revolute">
     <parent link="base_link"/>
     <child link="link2"/>
     <axis xyz="0 0 1"/>
     <origin xyz="0 0 ${link1_height}"/>
+    <limit effort="1000.0" lower="${-pi/2}" upper="${pi/2}" velocity="0.5"/>
   </joint>
-  <joint name="joint2" type="continuous">
+  <joint name="joint2" type="revolute">
     <parent link="link2"/>
     <child link="link3"/>
     <axis xyz="0 1 0"/>
     <origin xyz="0 0 ${link2_height}"/>
+    <limit effort="1000.0" lower="${-pi/2}" upper="${pi/2}" velocity="0.5"/>
   </joint>
-  <joint name="joint3" type="continuous">
+  <joint name="joint3" type="revolute">
     <parent link="link3"/>
     <child link="link4"/>
     <axis xyz="0 1 0"/>
     <origin xyz="0 0 ${link3_len}"/>
+    <limit effort="1000.0" lower="${-pi*0.48}" upper="${pi*0.75}" velocity="0.5"/>
   </joint>
-  <joint name="joint4" type="continuous">
+  <joint name="joint4" type="revolute">
     <parent link="link4"/>
     <child link="link5"/>
     <axis xyz="0 1 0"/>
     <origin xyz="0 0 ${link4_len}"/>
+    <limit effort="1000.0" lower="${-pi/2}" upper="${pi/2}" velocity="0.5"/>
   </joint>
-  <joint name="joint5" type="continuous">
+  <joint name="joint5" type="revolute">
     <parent link="link5"/>
     <child link="link6"/>
     <axis xyz="0 0 1"/>
     <origin xyz="0 0 ${link5_len / 2}"/>
+    <limit effort="1000.0" lower="${-pi/2}" upper="${pi/2}" velocity="0.5"/>
   </joint>
   <joint name="link6-tool0" type="fixed">
-  <parent link="link6" />
-  <child link="tool0" />
-  <origin xyz="0 0 ${link6_len}" rpy="0 -1.57075 0" />
-</joint>
+      <parent link="link6" />
+      <child link="tool0" />
+      <origin xyz="0 0 ${link6_len}" rpy="0 -1.57075 0" />
+    </joint>
+    <joint name="tool0_gripper" type="fixed">
+      <parent link="tool0" />
+      <child link="gripper_base" />
+      <origin xyz="0.0 0 0" rpy="0 0 0" />
+    </joint>
+  <joint name="gripper_joint" type="revolute">
+    <parent link="gripper_base"/>
+    <child link="gripper_link_left"/>
+    <axis xyz="0 0 1"/>
+    <origin xyz="-0.055 0.02 0"/>
+    <limit effort="1000.0" lower="0" upper="${gripper_open_angle}" velocity="0.5"/>
+  </joint>
+  <joint name="gripper_joint_right" type="revolute">
+    <mimic joint="gripper_joint" multiplier="-1"/>
+    <parent link="gripper_base"/>
+    <child link="gripper_link_right"/>
+    <axis xyz="0 0 1"/>
+    <origin xyz="-0.055 -0.02 0"/>
+    <limit effort="1000.0" lower="${gripper_open_angle}" upper="0" velocity="0.5"/>
+  </joint>
+    <link name="gripper_base">
+   </link>
+  <link name="gripper_link_left" >
+    <visual>
+      <geometry>
+        <box size="0.06 0.005 0.02"/>
+      </geometry>
+      <origin xyz="0.03 0 0"/>
+      <material name="orange"/>
+    </visual>
+  </link>
+  <link name="gripper_link_right" >
+    <visual>
+      <geometry>
+        <box size="0.06 0.005 0.02"/>
+      </geometry>
+      <origin xyz="0.03 0 0"/>
+      <material name="orange"/>
+    </visual>
+  </link>
 </robot>

Commit message: Arm v2 config and launch files
- files for the new v2 arm made from Feetech SCS215 servos
- Updated URDF and IK plugin
- updated arips_arm_node to control servos over serial
- some demo python scripts

File: arips_arm_description/urdf/arips_arm.urdf (robot description, URDF)
Before this commit: robot arips_arm, 9 links, 8 joints
Links:
- removed link gripper_link
- added link gripper_link_left; visual box size=0.06 0.005 0.02
- added link gripper_link_right; visual box size=0.06 0.005 0.02
- link link3: geometry visual box size=0.02 0.05 0.14
- link link5: geometry visual box size=0.01 0.04 0.035
- link link6: geometry visual cylinder length=0.045 radius=0.01
- link tool0: geometry visual box size=0.012 0.022 0.02
Joints:
- removed joint xgripper_joint
- added joint gripper_joint: type revolute, parent gripper_base, child gripper_link_left, origin xyz=-0.055 0.02 0, axis 0 0 1, limit lower=0 upper=0.3 effort=1000.0 velocity=1.0
- added joint gripper_joint_right: type revolute, parent gripper_base, child gripper_link_right, origin xyz=-0.055 -0.02 0, axis 0 0 1, limit lower=0.3 upper=0 effort=1000.0 velocity=1.0, mimic joint=gripper_joint multiplier=-1
- joint joint1: limit (none) -> lower=-1.41371669412 upper=1.41371669412 effort=1000.0 velocity=1.0; type continuous -> revolute
- joint joint2: limit (none) -> lower=-0.95 upper=2.1 effort=1000.0 velocity=1.0; origin xyz=0 0 0.07 -> xyz=0.02 0 0.07; type continuous -> revolute
- joint joint3: limit (none) -> lower=-1.50796447372 upper=3.0 effort=1000.0 velocity=1.0; origin xyz=0 0 0.12 -> xyz=0 0 0.14; type continuous -> revolute
- joint joint4: limit (none) -> lower=-1.5707963268 upper=1.5707963268 effort=1000.0 velocity=1.0; type continuous -> revolute
- joint joint5: limit (none) -> lower=-1.5707963268 upper=1.5707963268 effort=1000.0 velocity=1.0; origin xyz=0 0 0.015 -> xyz=0 0 0.0175; type continuous -> revolute
- joint link6-tool0: origin xyz=0 0 0.025 rpy=0 -1.57075 0 -> xyz=0 0 0.085 rpy=0 -1.57075 0
- joint tool0_gripper: origin xyz=0 0 0 rpy=0 0 0 -> xyz=0.0 0 0 rpy=0 0 0

File: arips_arm_description/urdf/arips_arm.xacro (robot description, xacro)
@@ -18,5 +18,5 @@
   <xacro:property name="link3_thick" value="0.02" />
   <xacro:property name="link3_width" value="0.05" />
-  <xacro:property name="link4_len" value="0.18" />
+  <xacro:property name="link4_len" value="0.15" />
   <xacro:property name="link4_thick" value="0.02" />
   <xacro:property name="link4_width" value="0.04" />
@@ -101,5 +101,5 @@
     <child link="link3"/>
     <axis xyz="0 1 0"/>
-    <origin xyz="0 0 ${link2_height}"/>
+    <origin xyz="0.02 0 ${link2_height}"/>
     <limit effort="1000.0" lower="-0.95" upper="2.1" velocity="1.0"/>
   </joint>

Commit message: Update MoveIt config, new launch files, calibration scripts

File: arips_arm_description/urdf/arips_arm.urdf (robot description, URDF)
Before this commit: robot arips_arm, 10 links, 9 joints
Joints:
- joint joint4: limit lower=-1.5707963268 upper=1.5707963268 effort=1000.0 velocity=1.0 -> lower=-1.57079632679 upper=1.57079632679 effort=1000.0 velocity=1.0
- joint joint5: limit lower=-1.5707963268 upper=1.5707963268 effort=1000.0 velocity=1.0 -> lower=-1.57079632679 upper=1.57079632679 effort=1000.0 velocity=1.0

File: arips_arm_description/urdf/arips_arm.xacro (robot description, xacro)
@@ -10,5 +10,4 @@
     <color rgba="1 0.6 0 1"/>
   </material>
-  <xacro:property name="pi" value="3.14159265359" />
   <xacro:property name="link1_sidelen" value="0.05" />
   <xacro:property name="link1_height" value="0.01" />

Commit message: pick_up left or right object user interaction handler, fixed arm_base_link in urdf#

File: arips_arm_description/urdf/arips_arm.urdf (robot description, URDF)
Before this commit: robot arips_arm, 10 links, 9 joints
Links:
- removed link base_link
- added link arm_base_link; visual box size=0.05 0.05 0.01
Joints:
- joint joint1: parent base_link -> arm_base_link
