Commit message: [arips_arm] Added gripper move group

File: arips_arm_description/urdf/arips_arm.xacro (robot description, xacro)
@@ -87,5 +87,5 @@
       </geometry>
       <origin xyz="-0.04 0 0.02"/>
-      <material name="orange"/>
+      <material name="black"/>
     </visual>
   </link>

Commit message: Better moveit setup, ground plane segmentation, pick and place demo

File: arips_arm_description/urdf/arips_arm.xacro (robot description, xacro)
@@ -15,8 +15,8 @@
   <xacro:property name="link2_height" value="0.07" />
   <xacro:property name="link2_radius" value="0.025" />
-  <xacro:property name="link3_len" value="0.12" />
+  <xacro:property name="link3_len" value="0.14" />
   <xacro:property name="link3_thick" value="0.02" />
   <xacro:property name="link3_width" value="0.05" />
-  <xacro:property name="link4_len" value="0.15" />
+  <xacro:property name="link4_len" value="0.18" />
   <xacro:property name="link4_thick" value="0.02" />
   <xacro:property name="link4_width" value="0.04" />
@@ -95,5 +95,5 @@
     <axis xyz="0 0 1"/>
     <origin xyz="0 0 ${link1_height}"/>
-    <limit effort="1000.0" lower="${-pi/2}" upper="${pi/2}" velocity="0.5"/>
+    <limit effort="1000.0" lower="${-pi*0.45}" upper="${pi*0.45}" velocity="1.0"/>
   </joint>
   <joint name="joint2" type="revolute">
@@ -102,5 +102,5 @@
     <axis xyz="0 1 0"/>
     <origin xyz="0 0 ${link2_height}"/>
-    <limit effort="1000.0" lower="${-pi/2}" upper="${pi/2}" velocity="0.5"/>
+    <limit effort="1000.0" lower="-0.95" upper="2.1" velocity="1.0"/>
   </joint>
   <joint name="joint3" type="revolute">
@@ -109,5 +109,5 @@
     <axis xyz="0 1 0"/>
     <origin xyz="0 0 ${link3_len}"/>
-    <limit effort="1000.0" lower="${-pi*0.48}" upper="${pi*0.75}" velocity="0.5"/>
+    <limit effort="1000.0" lower="${-pi*0.48}" upper="3.0" velocity="1.0"/>
   </joint>
   <joint name="joint4" type="revolute">
@@ -116,5 +116,5 @@
     <axis xyz="0 1 0"/>
     <origin xyz="0 0 ${link4_len}"/>
-    <limit effort="1000.0" lower="${-pi/2}" upper="${pi/2}" velocity="0.5"/>
+    <limit effort="1000.0" lower="${-pi/2}" upper="${pi/2}" velocity="1.0"/>
   </joint>
   <joint name="joint5" type="revolute">
@@ -123,5 +123,5 @@
     <axis xyz="0 0 1"/>
     <origin xyz="0 0 ${link5_len / 2}"/>
-    <limit effort="1000.0" lower="${-pi/2}" upper="${pi/2}" velocity="0.5"/>
+    <limit effort="1000.0" lower="${-pi/2}" upper="${pi/2}" velocity="1.0"/>
   </joint>
   <joint name="link6-tool0" type="fixed">
@@ -140,5 +140,5 @@
     <axis xyz="0 0 1"/>
     <origin xyz="-0.055 0.02 0"/>
-    <limit effort="1000.0" lower="0" upper="${gripper_open_angle}" velocity="0.5"/>
+    <limit effort="1000.0" lower="0" upper="${gripper_open_angle}" velocity="1.0"/>
   </joint>
   <joint name="gripper_joint_right" type="revolute">
@@ -148,5 +148,5 @@
     <axis xyz="0 0 1"/>
     <origin xyz="-0.055 -0.02 0"/>
-    <limit effort="1000.0" lower="${gripper_open_angle}" upper="0" velocity="0.5"/>
+    <limit effort="1000.0" lower="${gripper_open_angle}" upper="0" velocity="1.0"/>
   </joint>
     <link name="gripper_base">

Commit message: Updated arips_description to include arips arm, changed arm base link from 'base_link' to 'arm_base_link'

File: arips_arm_description/urdf/arips_arm.xacro (robot description, xacro)
@@ -26,5 +26,5 @@
   <xacro:property name="link6_radius" value="0.01" />
   <xacro:property name="gripper_open_angle" value="0.3" />
-  <link name="base_link">
+  <link name="arm_base_link">
   	<visual>
       <geometry>
@@ -90,5 +90,5 @@
   </link>
   <joint name="joint1" type="revolute">
-    <parent link="base_link"/>
+    <parent link="arm_base_link"/>
     <child link="link2"/>
     <axis xyz="0 0 1"/>

File: arips_description/urdf/arips.urdf (robot description, URDF)
Before this commit: robot arips, 4 links, 3 joints
Links:
- removed link arm_hand_link
- removed link arm_shoulder_link
- added link arm_base_link; visual box size=0.05 0.05 0.01
- added link gripper_base
- added link gripper_link_left; visual box size=0.06 0.005 0.02
- added link gripper_link_right; visual box size=0.06 0.005 0.02
- added link link2; visual cylinder length=0.07 radius=0.025
- added link link3; visual box size=0.02 0.05 0.14
- added link link4; visual box size=0.02 0.04 0.15
- added link link5; visual box size=0.01 0.04 0.035
- added link link6; visual cylinder length=0.045 radius=0.01
- added link tool0; visual box size=0.012 0.022 0.02
Joints:
- removed joint hand_joint
- removed joint shoulder_joint
- added joint base_to_right_leg: type fixed, parent base_link, child arm_base_link, origin xyz=0.163 -0.006 0.055 rpy=-0.028 0 0
- added joint gripper_joint: type revolute, parent gripper_base, child gripper_link_left, origin xyz=-0.055 0.02 0, axis 0 0 1, limit lower=0 upper=0.3 effort=1000.0 velocity=1.0
- added joint gripper_joint_right: type revolute, parent gripper_base, child gripper_link_right, origin xyz=-0.055 -0.02 0, axis 0 0 1, limit lower=0.3 upper=0 effort=1000.0 velocity=1.0, mimic joint=gripper_joint multiplier=-1
- added joint joint1: type revolute, parent arm_base_link, child link2, origin xyz=0 0 0.01, axis 0 0 1, limit lower=-1.41371669412 upper=1.41371669412 effort=1000.0 velocity=1.0
- added joint joint2: type revolute, parent link2, child link3, origin xyz=0.02 0 0.07, axis 0 1 0, limit lower=-0.95 upper=2.1 effort=1000.0 velocity=1.0
- added joint joint3: type revolute, parent link3, child link4, origin xyz=0 0 0.14, axis 0 1 0, limit lower=-1.50796447372 upper=3.0 effort=1000.0 velocity=1.0
- added joint joint4: type revolute, parent link4, child link5, origin xyz=0 0 0.15, axis 0 1 0, limit lower=-1.57079632679 upper=1.57079632679 effort=1000.0 velocity=1.0
- added joint joint5: type revolute, parent link5, child link6, origin xyz=0 0 0.0175, axis 0 0 1, limit lower=-1.57079632679 upper=1.57079632679 effort=1000.0 velocity=1.0
- added joint link6-tool0: type fixed, parent link6, child tool0, origin xyz=0 0 0.085 rpy=0 -1.57075 0
- added joint tool0_gripper: type fixed, parent tool0, child gripper_base, origin xyz=0.0 0 0 rpy=0 0 0

Commit message: localization capability, place object on object

File: arips_arm_description/urdf/arips_arm.xacro (robot description, xacro)
@@ -25,5 +25,5 @@
   <xacro:property name="link6_len" value="0.085" />
   <xacro:property name="link6_radius" value="0.01" />
-  <xacro:property name="gripper_open_angle" value="0.3" />
+  <xacro:property name="gripper_open_angle" value="0.06" />
   <link name="arm_base_link">
   	<visual>
@@ -108,5 +108,5 @@
     <axis xyz="0 1 0"/>
     <origin xyz="0 0 ${link3_len}"/>
-    <limit effort="1000.0" lower="${-pi*0.48}" upper="3.0" velocity="1.0"/>
+    <limit effort="1000.0" lower="${-pi*0.55}" upper="3.0" velocity="1.0"/>
   </joint>
   <joint name="joint4" type="revolute">
@@ -139,5 +139,5 @@
     <axis xyz="0 0 1"/>
     <origin xyz="-0.055 0.02 0"/>
-    <limit effort="1000.0" lower="0" upper="${gripper_open_angle}" velocity="1.0"/>
+    <limit effort="1000.0" lower="0.02" upper="${gripper_open_angle}" velocity="1.0"/>
   </joint>
   <joint name="gripper_joint_right" type="revolute">
@@ -147,5 +147,5 @@
     <axis xyz="0 0 1"/>
     <origin xyz="-0.055 -0.02 0"/>
-    <limit effort="1000.0" lower="${gripper_open_angle}" upper="0" velocity="1.0"/>
+    <limit effort="1000.0" lower="${gripper_open_angle}" upper="0.02" velocity="1.0"/>
   </joint>
     <link name="gripper_base">
